File: PCBs/Flex_oxymeter/oxymeter.kicad_sch (KiCad schematic)
At the start: 4 parts, among them J1 Conn_01x06_Pin, U1 MAX30102

Commit message: Add progress report for 31.1.2025 Update relevant source files
Other:
- title: (none) -> Oxymeter
Changed lines of the file:
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@@
 	(generator_version "8.0")
 	(paper "A4")
+	(title_block
+		(title "Oxymeter")
+	)
 	(junction
 		(at 72.39 93.98)
@@
 	(label "SCL"
 		(at 58.42 88.9 0)
-		(fields_autoplaced yes)
 		(effects
 			(font
@@
 	(label "+1V8"
 		(at 58.42 86.36 0)
-		(fields_autoplaced yes)
 		(effects
 			(font
@@
 	(label "GND"
 		(at 58.42 93.98 0)
-		(fields_autoplaced yes)
 		(effects
 			(font
@@
 	(label "INT"
 		(at 57.15 97.79 270)
-		(fields_autoplaced yes)
 		(effects
 			(font
@@
 	(label "SDA"
 		(at 58.42 91.44 0)
-		(fields_autoplaced yes)
 		(effects
 			(font
@@
 	(label "+3V3"
 		(at 58.42 83.82 0)
-		(fields_autoplaced yes)
-		(effects
-			(font
+		(effects
+			(font
