File: PCBs/Flex_pogo_female/pogo_female.kicad_sch (KiCad schematic)
At the start: 2 parts, among them J1 Pogo pads, J2 Conn_01x04_Pin

Commit message: Add progress report for 31.1.2025 Update relevant source files
Other:
- title: (none) -> Female flex pogo pin USB connector (for watch)
Changed lines of the file:
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@@
 	(generator_version "8.0")
 	(paper "A4")
+	(title_block
+		(title "Female flex pogo pin USB connector (for watch)")
+	)
 	(wire
 		(pts
@@
 	(label "+5V"
 		(at 168.91 92.71 0)
-		(fields_autoplaced yes)
 		(effects
 			(font
@@
 	(label "GND"
 		(at 168.91 100.33 0)
-		(fields_autoplaced yes)
 		(effects
 			(font
@@
 	(label "D-"
 		(at 168.91 95.25 0)
-		(fields_autoplaced yes)
 		(effects
 			(font
@@
 	(label "D+"
 		(at 168.91 97.79 0)
-		(fields_autoplaced yes)
 		(effects
 			(font
