File: PCBs/Mainboard/display.kicad_sch (KiCad schematic)
At the start: 9 parts, among them J5 Conn_02x12_Counter_Clockwise_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, U4 TPS65136RTER

Commit message: Add progress report for 31.1.2025 Update relevant source files
Other:
- note removed: "Schematic IO-expander"
- title: (none) -> Display
Changed lines of the file:
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@@
 	(generator_version "8.0")
 	(paper "A4")
+	(title_block
+		(title "Display")
+	)
 	(junction
 		(at 237.49 44.45)
@@
 		)
 	)
-	(text "Schematic IO-expander"
-		(exclude_from_sim no)
-		(at 202.692 189.738 0)
-		(effects
-			(font
-				(size 1.778 1.778)
-			)
-		)
-	)
 	(label "ELVSS"
 		(at 262.89 86.36 180)
-		(fields_autoplaced yes)
 		(effects
 			(font
@@
 	(label "SWIRE"
 		(at 125.73 81.28 0)
-		(fields_autoplaced yes)
 		(effects
 			(font
@@
 	(label "FB"
 		(at 224.79 44.45 0)
-		(fields_autoplaced yes)
 		(effects
 			(font
@@
 	(label "ELVSS"
 		(at 125.73 66.04 0)
-		(fields_autoplaced yes)
 		(effects
 			(font
@@
 	(label "ELVDD"
 		(at 224.79 41.91 0)
-		(fields_autoplaced yes)
 		(effects
 			(font
@@
 	(label "FBG"
 		(at 224.79 57.15 0)
-		(fields_autoplaced yes)
 		(effects
 			(font
@@
 	(label "FBG"
 		(at 125.73 76.2 0)
-		(fields_autoplaced yes)
 		(effects
 			(font
@@
 	(label "ELVDD"
 		(at 59.69 58.42 180)
-		(fields_autoplaced yes)
 		(effects
 			(font
@@
 	(label "ELVSS"
 		(at 224.79 69.85 0)
-		(fields_autoplaced yes)
 		(effects
 			(font
@@
 	(label "ELVDD"
 		(at 224.79 86.36 0)
-		(fields_autoplaced yes)
 		(effects
 			(font
@@
 	(label "ELVSS"
 		(at 59.69 55.88 180)
-		(fields_autoplaced yes)
 		(effects
 			(font
@@
 	(label "FB"
 		(at 125.73 78.74 0)
-		(fields_autoplaced yes)
 		(effects
 			(font
@@
 	(label "ELVDD"
 		(at 207.01 81.28 180)
-		(fields_autoplaced yes)
 		(effects
 			(font
@@
 	(label "SWIRE"
 		(at 59.69 71.12 180)
-		(fields_autoplaced yes)
 		(effects
 			(font
@@
 		(shape input)
 		(at 50.8 73.66 0)
-		(fields_autoplaced yes)
 		(effects
 			(font
@@
 		(shape input)
 		(at 50.8 76.2 0)
-		(fields_autoplaced yes)
 		(effects
 			(font
@@
 		(shape input)
 		(at 38.1 63.5 180)
-		(fields_autoplaced yes)
 		(effects
 			(font
@@
 		(shape input)
 		(at 38.1 78.74 180)
-		(fields_autoplaced yes)
 		(effects
 			(font
@@
 		(shape input)
 		(at 38.1 73.66 180)
-		(fields_autoplaced yes)
 		(effects
 			(font
@@
 		(shape input)
 		(at 38.1 58.42 180)
-		(fields_autoplaced yes)
 		(effects
 			(font
@@
 		(shape input)
 		(at 38.1 68.58 180)
-		(fields_autoplaced yes)
 		(effects
 			(font
@@
 		(shape input)
 		(at 50.8 81.28 0)
-		(fields_autoplaced yes)
 		(effects
 			(font
@@
 		(shape input)
 		(at 38.1 60.96 180)
-		(fields_autoplaced yes)
 		(effects
 			(font
@@
 		(shape input)
 		(at 50.8 78.74 0)
-		(fields_autoplaced yes)
 		(effects
 			(font
@@
 		(shape input)
 		(at 38.1 55.88 180)
-		(fields_autoplaced yes)
 		(effects
 			(font
@@
 		(shape input)
 		(at 95.25 63.5 180)
-		(fields_autoplaced yes)
 		(effects
 			(font
@@
 		(shape input)
 		(at 38.1 71.12 180)
-		(fields_autoplaced yes)
-		(effects
-			(font
+		(effects
+			(font
