File: PCBs/Mainboard/imu.kicad_sch (KiCad schematic)
At the start: 4 parts, among them IC1 ICM-42670-P

Commit message: Add progress report for 31.1.2025 Update relevant source files
Other:
- note removed: "Schematic IMU"
- title: (none) -> Battery IC & Step-down
Changed lines of the file:
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@@
 	(generator_version "8.0")
 	(paper "A4")
+	(title_block
+		(title "Battery IC & Step-down")
+	)
 	(junction
 		(at 101.6 113.03)
@@
 		)
 	)
-	(text "Schematic IMU"
-		(exclude_from_sim no)
-		(at 196.596 189.992 0)
-		(effects
-			(font
-				(size 1.778 1.778)
-			)
-		)
-	)
 	(hierarchical_label "INT1"
 		(shape input)
 		(at 71.12 82.55 180)
-		(fields_autoplaced yes)
 		(effects
 			(font
@@
 		(shape input)
 		(at 97.79 26.67 180)
-		(fields_autoplaced yes)
 		(effects
 			(font
@@
 		(shape input)
 		(at 97.79 22.86 180)
-		(fields_autoplaced yes)
 		(effects
 			(font
@@
 		(shape input)
 		(at 71.12 74.93 180)
-		(fields_autoplaced yes)
 		(effects
 			(font
@@
 		(shape input)
 		(at 127 80.01 0)
-		(fields_autoplaced yes)
-		(effects
-			(font
+		(effects
+			(font
