File: PCBs/Mainboard/vibro_ic.kicad_sch (KiCad schematic)
At the start: 3 parts, among them IC6 DA7280-00FV2, J8 vibro

Commit message: Add progress report for 31.1.2025 Update relevant source files
Other:
- title: (none) -> LRA Driver (Vibration)
Changed lines of the file:
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@@
 	(generator_version "8.0")
 	(paper "A4")
+	(title_block
+		(title "LRA Driver (Vibration)")
+	)
 	(junction
 		(at 54.61 81.28)
@@
 		(shape input)
 		(at 54.61 99.06 90)
-		(fields_autoplaced yes)
 		(effects
 			(font
@@
 		(shape input)
 		(at 72.39 60.96 90)
-		(fields_autoplaced yes)
 		(effects
 			(font
@@
 		(shape input)
 		(at 74.93 60.96 90)
-		(fields_autoplaced yes)
 		(effects
 			(font
@@
 		(shape input)
 		(at 77.47 60.96 90)
-		(fields_autoplaced yes)
 		(effects
 			(font
