File: PCBs/pogo_male/pogo_male.kicad_sch (KiCad schematic)
At the start: 6 parts, among them J1 USB_C_Receptacle_USB2.0_16P, J2 Conn_01x04_Pin

Commit message: Add progress report for 31.1.2025 Update relevant source files
Other:
- title: (none) -> Male pogo pin USB connector (for charging "case")
Changed lines of the file:
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@@
 	(generator_version "8.0")
 	(paper "A4")
+	(title_block
+		(title "Male pogo pin USB connector (for charging \"case\")")
+	)
 	(junction
 		(at 95.25 80.01)
@@
 	(label "D+"
 		(at 99.06 80.01 0)
-		(fields_autoplaced yes)
 		(effects
 			(font
@@
 	(label "D+"
 		(at 161.29 82.55 180)
-		(fields_autoplaced yes)
 		(effects
 			(font
@@
 	(label "D-"
 		(at 99.06 85.09 0)
-		(fields_autoplaced yes)
 		(effects
 			(font
@@
 	(label "GND"
 		(at 161.29 87.63 180)
-		(fields_autoplaced yes)
 		(effects
 			(font
@@
 	(label "D-"
 		(at 161.29 85.09 180)
-		(fields_autoplaced yes)
 		(effects
 			(font
@@
 	(label "+5V"
 		(at 95.25 66.04 0)
-		(fields_autoplaced yes)
 		(effects
 			(font
@@
 	(label "+5V"
 		(at 161.29 80.01 180)
-		(fields_autoplaced yes)
-		(effects
-			(font
+		(effects
+			(font
